File: PCB/PCB Design.brd (EAGLE design)
At the start: 46 x 41.9 mm, 17 parts, among them Q1 16MHz

Commit message: Added diode and rtc
Parts:
- added D1, D2: 250mA/100V, SparkFun-DiscreteSemi:SOD-323
- added JP4: (no value), pinhead:1X05
- added R1: 10k, resistor:M0805
- moved R3 22.7 mm to (43.2, 15.2)
- moved C8 21.9 mm to (39.4, 19.1)
- moved C2 6.82 mm to (18.4, 21.2), turned to 180 degrees
- moved C6 6.59 mm to (32.5, 11.3)
- moved C5 5.75 mm to (27.9, 11.3)
- moved C4 2.57 mm to (18.7, 26.2), turned to 180 degrees
- moved PIR 1.91 mm to (29.6, 5.08), turned to 0 degrees
Connections:
- new net 8: D2.A, NRF1.8
- new net N$6: D1.A, JP4.5
- net GND: now also JP4.1, R1.1
- net PC3/A3: now also JP4.2
- net PC4/A4/SDA: now also JP4.3
- net PC5/A5/SCL: now also JP4.4
- net PD2/INT0: now also D1.C, D2.C, R1.2; no longer NRF1.8
Routing:
- net PD2/INT0: track 49.7 -> 8.14 mm, vias 3 -> 0
- net 8: track 0.00 -> 38.2 mm, vias 0 -> 1
- net PC3/A3: track 0.00 -> 22.1 mm, vias 0 -> 1
- net PC4/A4/SDA: track 0.00 -> 18.6 mm, vias 0 -> 1
- net PC5/A5/SCL: track 0.00 -> 15.1 mm, vias 0 -> 1
- net V+: track 24.8 -> 32.6 mm
- net N$6: track 0.00 -> 6.79 mm, vias 0 -> 1
- net DTR: track 18.1 -> 12.8 mm
- net PC6/RESET: track 69.2 -> 73.3 mm, vias 1 -> 2
- net PD0/RX: track 18.0 -> 14.5 mm, vias 2 -> 0
- net PB2/D10/CE: track 17.7 -> 14.8 mm
- net PD3/INT1: track 19.6 -> 21.5 mm
- net PD1/TX: track 14.4 -> 13.0 mm
- net PB6/CRYSTAL1: track 13.7 -> 13.0 mm
- net PD6: track 13.1 -> 12.4 mm
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Other:
- board text removed: "5V"
- board text removed: "CTS"
- board text removed: "DTR"
- board text removed: "RX"
- board text removed: "TX"

Commit message: Generated Gerbers
Parts:
- removed 1117: V_REG_LD1117VXXLD1117-SMD, SparkFun-IC-Power:SOT223
- added C1: .1uF, rcl:C0805K
- added C3: 1uf, rcl:E2,5-5
- added C7: 470pF, rcl:C0805K
- added U2: TC1014, SparkFun-IC-Power:SOT23-5
- C8: value 10uf -> 1uf; device resistor:E2,5-6 -> rcl:E2,5-5
- Q1: value 16MHz -> 8MHz
- moved JP2 4.89 mm to (49.4, 1.78), turned to 180 degrees
- moved RESET 3.07 mm to (39.4, 6.48), turned to 180 degrees
- moved PIR 2.03 mm to (29.6, 3.05)
- moved JP1 1.99 mm to (49.4, 5.33), turned to 0 degrees
- moved C2 0.81 mm to (18.9, 20.6), turned to 90 degrees
- moved C6 0.76 mm to (33.3, 11.3)
- moved JP4 0.25 mm to (18.2, 15.9), turned to 180 degrees
- renumbered NRF1 to NRF, OLED1 to OLED
Connections:
- new net BYPASS: C7.1, U2.4
- net +3V3: now also C1.1, PIR.1, U2.5; no longer 1117.2
- net GND: now also C1.2, C3.-, C7.2, U2.2; no longer 1117.1
- net V+: now also C3.+, U2.1, U2.3; no longer 1117.3, PIR.1
Routing:
- net +3V3: track 110.4 -> 142.3 mm, vias 4 -> 5
- net N$6: track 6.79 -> 22.2 mm
- net V+: track 32.6 -> 19.7 mm
- net PC3/A3: track 22.1 -> 16.4 mm
- net BYPASS: track 0.00 -> 5.53 mm
- net PC5/A5/SCL: track 15.1 -> 19.5 mm
- net PB3/MOSI/D11: track 66.3 -> 62.2 mm, vias 5 -> 3
- net PD5/CSN: track 37.5 -> 41.4 mm
- net PD3/INT1: track 21.5 -> 23.6 mm
- net PC6/RESET: track 73.3 -> 71.6 mm, vias 2 -> 4
- net PC4/A4/SDA: track 18.6 -> 17.8 mm
Other:
- board size 46 x 41.9 mm -> 46 x 44.8 mm
- board text added: "Chirag Shah Srijal Poojari 2/Apr/18"
- board text added: "Room Occupancy System"
